Commit message: play.py works with xbot+gazebo

File: src/jumping_leg/models/red_intangible_ball.urdf.xacro (robot description, xacro)
@@ -14,5 +14,4 @@
 		</inertial>
 	</xacro:macro>
-    <link name="world"/>
 	<link name="sphere_link">
 		<!-- The shin is made of a cylinder plus a sphere, the total length, is shin_height, so the length  of the two are detemrined accordingly -->
@@ -38,7 +37,3 @@
       	</visual>
     </gazebo>
-	<joint name="world_to_sphere" type="fixed">
-        <parent link="world"/>
-        <child link="sphere_link"/>
-    </joint>
 </robot>

File: src/jumping_leg/models/support.urdf.xacro (robot description, xacro)
@@ -18,6 +18,6 @@
 		</inertial>
 	</xacro:macro>
-    <link name="world"/>
-	<link name="box_link">
+    <!-- <link name="world"/> -->
+	<link name="plate">
 		<!-- The shin is made of a cylinder plus a sphere, the total length, is shin_height, so the length  of the two are detemrined accordingly -->
         <visual>
@@ -61,5 +61,5 @@
 			</contact>
 	</link>
-	<gazebo reference="box_link">
+	<gazebo reference="plate">
 		<visual name="visual">
 			<material>
@@ -73,7 +73,3 @@
       	</visual>
     </gazebo>
-	<joint name="world_to_sphere" type="fixed">
-        <parent link="world"/>
-        <child link="box_link"/>
-    </joint>
 </robot>
