Commit message: added slider

File: src/jumping_leg/models/leg_simple.urdf.xacro (robot description, xacro)
@@ -17,4 +17,9 @@
 	<xacro:arg name="rail_height" default="2" />
 	<xacro:arg name="rail_mass" default="1000" />
+	<xacro:arg name="slider_width" default="0.15" />
+	<xacro:arg name="slider_length" default="0.01" />
+	<xacro:arg name="slider_height" default="0.15" />
+	<xacro:arg name="slider_y_offset" default="0.01" />
+	<xacro:arg name="slider_mass" default="8" />
 	<xacro:arg name="hip_friction" default="0.1" />
 	<xacro:arg name="rail_friction" default="0.0" />
@@ -41,4 +46,9 @@
 	<xacro:property name="rail_height" default="$(arg rail_height)" />
 	<xacro:property name="rail_mass" default="$(arg rail_mass)" />
+	<xacro:property name="slider_width" default="$(arg slider_width)" />
+	<xacro:property name="slider_length" default="$(arg slider_length)" />
+	<xacro:property name="slider_height" default="$(arg slider_height)" />
+	<xacro:property name="slider_mass" default="$(arg slider_mass)" />
+	<xacro:property name="slider_y_offset" default="$(arg slider_y_offset)" />
 	<xacro:property name="knee_friction" default="$(arg knee_friction)" />
 	<xacro:property name="hip_friction" default="$(arg hip_friction)" />
@@ -109,5 +119,22 @@
       	</visual>
     </gazebo>
-    <link name="slider_link"/>
+    <link name="slider_link">
+		<visual name = "slider_link_v">
+			<origin xyz="0 ${slider_y_offset} 0" rpy="0 0 0"/>
+			<geometry>
+				<box size="${slider_width} ${slider_length} ${slider_height}"/>
+			</geometry>
+	   	</visual>
+  		<collision name = "slider_link_c">
+			<origin xyz="0 ${slider_y_offset} 0" rpy="0 0 0"/>
+			<geometry>
+				<box size="${slider_width} ${slider_length} ${slider_height}"/>
+			</geometry>
+	   	</collision>
+		<xacro:box_inertial mass="${slider_mass}"
+                            x="${slider_width}" y="${slider_length}" z="${slider_height}"
+                            pose_xyz = "0 0 ${slider_height}"
+                            pose_rpy = "0 0 0"/>
+	</link>
 	<link name="thigh_link">
 		<visual name = "thigh_link_v">

Commit message: testing energy diff reward

File: src/jumping_leg/models/leg_simple.urdf.xacro (robot description, xacro)
@@ -152,4 +152,5 @@
 		<xacro:cylinder_z_inertial mass="${thigh_mass}" height="${thigh_height}" radius="${thigh_width/2}" pose_xyz="0 0 -${thigh_height/2}" pose_rpy="0 0 0"/>
 	</link>
+	<link name="thigh_link_base"/>
 	<gazebo reference="thigh_link">
 		<visual name="thigh_link_v">
@@ -192,4 +193,5 @@
 		<xacro:cylinder_z_inertial mass="${shin_mass}" height="${shin_height}" radius="${shin_width/2}" pose_xyz="0 0 -${shin_height/2}" pose_rpy="0 0 0"/>
 	</link>
+	<link name="shin_link_base"/>
 	<gazebo reference="shin_link">
 		<visual name="visual">
@@ -224,4 +226,8 @@
         <axis xyz="0 1 0"/>
 	</joint>
+	<joint name="thigh_link_base" type="fixed">
+        <parent link="thigh_link"/>
+        <child link="thigh_link_base"/>
+    </joint>
  	<joint name="knee_joint" type="revolute">
     	<parent link="thigh_link"/>
@@ -232,4 +238,8 @@
         <axis xyz="0 1 0"/>
 	</joint>
+	<joint name="shin_link_base" type="fixed">
+        <parent link="shin_link"/>
+        <child link="shin_link_base"/>
+    </joint>
 	<joint name="foot_joint" type="fixed">
         <parent link="shin_link"/>

Commit message: starting to work nice

File: src/jumping_leg/models/leg_simple.urdf.xacro (robot description, xacro)
@@ -152,5 +152,10 @@
 		<xacro:cylinder_z_inertial mass="${thigh_mass}" height="${thigh_height}" radius="${thigh_width/2}" pose_xyz="0 0 -${thigh_height/2}" pose_rpy="0 0 0"/>
 	</link>
-	<link name="thigh_link_base"/>
+	<link name="thigh_link_base">
+		<xacro:box_inertial mass="0.0001"
+                            x="0.001" y="0.001" z="0.001"
+                            pose_xyz = "0 0 0"
+                            pose_rpy = "0 0 0"/>
+	</link>
 	<gazebo reference="thigh_link">
 		<visual name="thigh_link_v">
@@ -192,6 +197,36 @@
         </collision>
 		<xacro:cylinder_z_inertial mass="${shin_mass}" height="${shin_height}" radius="${shin_width/2}" pose_xyz="0 0 -${shin_height/2}" pose_rpy="0 0 0"/>
-	</link>
-	<link name="shin_link_base"/>
+		<contact>
+				<!--
+				Pybullet defaults maybe are these (from bullet3/examples/Importers/ImportURDFDemo/URDFJointTypes.h line 33)
+				URDFLinkContactInfo()
+					: m_lateralFriction(0.5),
+					m_rollingFriction(0),
+					m_spinningFriction(0),
+					m_restitution(0),
+					m_inertiaScaling(1),
+					m_contactCfm(0),
+					m_contactErp(0),
+					m_contactStiffness(1e4),
+					m_contactDamping(1)
+				-->
+				<lateral_friction value="0.9"/>
+				<rolling_friction value="0.01"/>
+				<!-- <contact_cfm value="0.1 "/> -->
+				<!-- <contact_erp value="0.2"/> -->
+				<restitution value="0.05"/>
+				<!-- <spinning_friction value="0"/> -->
+				<!-- <friction_anchor value="0"/> -->
+				<!-- <inertia_scaling value="0"/> -->
+				<!-- <stiffness value="2500"/> -->
+				<!-- <damping value="8"/>  -->
+			</contact>
+	</link>
+	<link name="shin_link_base">
+		<xacro:box_inertial mass="0.0001"
+                            x="0.001" y="0.001" z="0.001"
+                            pose_xyz = "0 0 0"
+                            pose_rpy = "0 0 0"/>
+	</link>
 	<gazebo reference="shin_link">
 		<visual name="visual">
@@ -206,5 +241,10 @@
       	</visual>
     </gazebo>
-    <link name="foot_link"/>
+    <link name="foot_link">
+		<xacro:box_inertial mass="0.0001"
+                            x="0.001" y="0.001" z="0.001"
+                            pose_xyz = "0 0 0"
+                            pose_rpy = "0 0 0"/>
+	</link>
 	<joint name="world_to_rail" type="fixed">
         <parent link="world"/>

File: src/jumping_leg/models/support.urdf.xacro (robot description, xacro)
@@ -35,4 +35,29 @@
         </collision>
 		<xacro:box_inertial mass="0.001" x="${size_x}" y="${size_y}" z="${size_z}" pose_xyz="0 0 0" pose_rpy="0 0 0"/>
+		<contact>
+				<!--
+				Pybullet defaults maybe are these (from bullet3/examples/Importers/ImportURDFDemo/URDFJointTypes.h line 33)
+				URDFLinkContactInfo()
+					: m_lateralFriction(0.5),
+					m_rollingFriction(0),
+					m_spinningFriction(0),
+					m_restitution(0),
+					m_inertiaScaling(1),
+					m_contactCfm(0),
+					m_contactErp(0),
+					m_contactStiffness(1e4),
+					m_contactDamping(1)
+				-->
+				<lateral_friction value="0.9"/>
+				<rolling_friction value="0.01"/>
+				<!-- <contact_cfm value="0.1 "/> -->
+				<!-- <contact_erp value="0.2"/> -->
+				<restitution value="0.05"/>
+				<!-- <spinning_friction value="0"/> -->
+				<!-- <friction_anchor value="0"/> -->
+				<!-- <inertia_scaling value="0"/> -->
+				<!-- <stiffness value="2500"/> -->
+				<!-- <damping value="8"/>  -->
+			</contact>
 	</link>
 	<gazebo reference="box_link">

Commit message: Configuration observation, frame stacking, somethign wrong with joint limits

File: src/jumping_leg/models/leg_simple.urdf.xacro (robot description, xacro)
@@ -171,5 +171,5 @@
     </gazebo>
 	<link name="shin_link">
-		<!-- The shin is made of a cylinder plus a sphere, the total length, is shin_height, so the length  of the two are detemrined accordingly -->
+		<!-- shin_height is the knee to foot tip distance, so the actual shin lenght is determined accordingly-->
 		<visual name = "shin_link_v">
 			<origin xyz="0 0 -${(shin_height-shin_width)/2}" rpy="0 0 0"/>
@@ -178,23 +178,72 @@
 			</geometry>
 	   </visual>
+		<collision name = "shin_link_c">
+			<origin xyz="0 0 -${(shin_height-shin_width)/2}" rpy="0 0 0"/>
+			<geometry>
+                <cylinder length="${shin_height-shin_width}" radius="${shin_width/2}" />
+			</geometry>
+	   </collision>
+		<xacro:cylinder_z_inertial mass="${shin_mass}" height="${shin_height}" radius="${shin_width/2}" pose_xyz="0 0 -${shin_height/2}" pose_rpy="0 0 0"/>
+		<contact>
+				<!--
+				Pybullet defaults maybe are these (from bullet3/examples/Importers/ImportURDFDemo/URDFJointTypes.h line 33)
+				URDFLinkContactInfo()
+					: m_lateralFriction(0.5),
+					m_rollingFriction(0),
+					m_spinningFriction(0),
+					m_restitution(0),
+					m_inertiaScaling(1),
+					m_contactCfm(0),
+					m_contactErp(0),
+					m_contactStiffness(1e4),
+					m_contactDamping(1)
+				-->
+				<lateral_friction value="0.05"/>
+				<rolling_friction value="0.01"/>
+				<!-- <contact_cfm value="0.1 "/> -->
+				<!-- <contact_erp value="0.2"/> -->
+				<restitution value="0.05"/>
+				<!-- <spinning_friction value="0"/> -->
+				<!-- <friction_anchor value="0"/> -->
+				<!-- <inertia_scaling value="0"/> -->
+				<!-- <stiffness value="2500"/> -->
+				<!-- <damping value="8"/>  -->
+			</contact>
+	</link>
+	<link name="shin_link_base">
+		<xacro:box_inertial mass="0.0001"
+                            x="0.001" y="0.001" z="0.001"
+                            pose_xyz = "0 0 0"
+                            pose_rpy = "0 0 0"/>
+	</link>
+	<gazebo reference="shin_link">
+		<visual name="visual">
+			<material>
+			<ambient>$(arg shin_color)</ambient>
+			<diffuse>$(arg shin_color)</diffuse>
+			<!--
+			<specular>1 0 0 1</specular>
+			<emissive>1 0 0 1</emissive>
+			-->
+			</material>
+      	</visual>
+    </gazebo>
+    <link name="foot_center_link">
         <visual>
-			<origin xyz="0 0 -${shin_height-shin_width}" rpy="0 0 0"/>
+			<origin xyz="0 0 0" rpy="0 0 0"/>
             <geometry>
                 <sphere radius="${shin_width}" />
             </geometry>
         </visual>
-		<collision name = "shin_link_c">
-			<origin xyz="0 0 -${(shin_height-shin_width)/2}" rpy="0 0 0"/>
-			<geometry>
-                <cylinder length="${shin_height-shin_width}" radius="${shin_width/2}" />
-			</geometry>
-	   </collision>
         <collision>
-			<origin xyz="0 0 -${shin_height-shin_width}" rpy="0 0 0"/>
+			<origin xyz="0 0 0" rpy="0 0 0"/>
             <geometry>
                 <sphere radius="${shin_width}" />
             </geometry>
         </collision>
-		<xacro:cylinder_z_inertial mass="${shin_mass}" height="${shin_height}" radius="${shin_width/2}" pose_xyz="0 0 -${shin_height/2}" pose_rpy="0 0 0"/>
+		<xacro:box_inertial mass="0.0001"
+                            x="0.001" y="0.001" z="0.001"
+                            pose_xyz = "0 0 0"
+                            pose_rpy = "0 0 0"/>
 		<contact>
 				<!--
@@ -223,22 +272,4 @@
 			</contact>
 	</link>
-	<link name="shin_link_base">
-		<xacro:box_inertial mass="0.0001"
-                            x="0.001" y="0.001" z="0.001"
-                            pose_xyz = "0 0 0"
-                            pose_rpy = "0 0 0"/>
-	</link>
-	<gazebo reference="shin_link">
-		<visual name="visual">
-			<material>
-			<ambient>$(arg shin_color)</ambient>
-			<diffuse>$(arg shin_color)</diffuse>
-			<!--
-			<specular>1 0 0 1</specular>
-			<emissive>1 0 0 1</emissive>
-			-->
-			</material>
-      	</visual>
-    </gazebo>
     <link name="foot_link">
 		<xacro:box_inertial mass="0.0001"
@@ -282,4 +313,9 @@
         <child link="shin_link_base"/>
     </joint>
+	<joint name="foot_center_joint" type="fixed">
+        <parent link="shin_link"/>
+        <child link="foot_center_link"/>
+    	<origin xyz="0 0 -${shin_height-shin_width}" rpy="0 0 0"/>
+    </joint>
 	<joint name="foot_joint" type="fixed">
         <parent link="shin_link"/>

File: src/jumping_leg/models/support.urdf.xacro (robot description, xacro)
@@ -3,5 +3,5 @@
 	<xacro:arg name="size_x" default="0.20" />
 	<xacro:arg name="size_y" default="0.50" />
-	<xacro:arg name="size_z" default="0.025" />
+	<xacro:arg name="size_z" default="0.005" />
 	<xacro:property name="size_x" default="$(arg size_x)" />
 	<xacro:property name="size_y" default="$(arg size_y)" />

Commit message: play works with rosxbotadapter

File: src/jumping_leg/models/leg_simple.urdf.xacro (robot description, xacro)
@@ -70,4 +70,10 @@
 		</inertial>
 	</xacro:macro>
+    <xacro:macro name="small_inertial" params="">
+		<xacro:box_inertial mass="0.0001"
+                            x="0.001" y="0.001" z="0.001"
+                            pose_xyz = "0 0 0"
+                            pose_rpy = "0 0 0"/>
+    </xacro:macro>
     <xacro:macro name="cylinder_z_inertial" params="mass height radius pose_xyz pose_rpy">
 		<inertial>
@@ -137,5 +143,5 @@
                             pose_rpy = "0 0 0"/>
 	</link>
-	<link name="thigh_link">
+	<link name="thigh_link_base">
 		<visual name = "thigh_link_v">
 			<origin xyz="0 0 -${thigh_height/2}" rpy="0 0 0"/>
@@ -143,5 +149,5 @@
                 <cylinder length="${thigh_height}" radius="${thigh_width/2}" />
 			</geometry>
-	   </visual>
+	   	</visual>
 		<collision name = "thigh_link_c">
 			<origin xyz="0 0 -${thigh_height/2}" rpy="0 0 0"/>
@@ -149,14 +155,12 @@
                 <cylinder length="${thigh_height}" radius="${thigh_width/2}" />
 			</geometry>
-	   </collision>
-		<xacro:cylinder_z_inertial mass="${thigh_mass}" height="${thigh_height}" radius="${thigh_width/2}" pose_xyz="0 0 -${thigh_height/2}" pose_rpy="0 0 0"/>
-	</link>
-	<link name="thigh_link_base">
-		<xacro:box_inertial mass="0.0001"
-                            x="0.001" y="0.001" z="0.001"
-                            pose_xyz = "0 0 0"
-                            pose_rpy = "0 0 0"/>
-	</link>
-	<gazebo reference="thigh_link">
+	   	</collision>
+		<xacro:small_inertial />
+	</link>
+	<link name="thigh_link_com">
+		<xacro:cylinder_z_inertial mass="${thigh_mass}" height="${thigh_height}" radius="${thigh_width/2}"
+									pose_xyz="0 0 0" pose_rpy="0 0 0"/>
+	</link>
+	<gazebo reference="thigh_link_base">
 		<visual name="thigh_link_v">
 			<material>
@@ -170,5 +174,5 @@
       	</visual>
     </gazebo>
-	<link name="shin_link">
+	<link name="shin_link_base">
 		<!-- shin_height is the knee to foot tip distance, so the actual shin lenght is determined accordingly-->
 		<visual name = "shin_link_v">
@@ -177,5 +181,5 @@
                 <cylinder length="${shin_height-shin_width}" radius="${shin_width/2}" />
 			</geometry>
-	   </visual>
+	   	</visual>
 		<collision name = "shin_link_c">
 			<origin xyz="0 0 -${(shin_height-shin_width)/2}" rpy="0 0 0"/>
@@ -183,6 +187,6 @@
                 <cylinder length="${shin_height-shin_width}" radius="${shin_width/2}" />
 			</geometry>
-	   </collision>
-		<xacro:cylinder_z_inertial mass="${shin_mass}" height="${shin_height}" radius="${shin_width/2}" pose_xyz="0 0 -${shin_height/2}" pose_rpy="0 0 0"/>
+		</collision>
+		<xacro:small_inertial />
 		<contact>
 				<!--
@@ -211,11 +215,9 @@
 			</contact>
 	</link>
-	<link name="shin_link_base">
-		<xacro:box_inertial mass="0.0001"
-                            x="0.001" y="0.001" z="0.001"
-                            pose_xyz = "0 0 0"
-                            pose_rpy = "0 0 0"/>
-	</link>
-	<gazebo reference="shin_link">
+	<link name="shin_link_com">
+		<xacro:cylinder_z_inertial mass="${shin_mass}" height="${shin_height}" radius="${shin_width/2}"
+									pose_xyz="0 0 -${shin_height/2}" pose_rpy="0 0 0"/>
+	</link>
+	<gazebo reference="shin_link_base">
 		<visual name="visual">
 			<material>
@@ -242,8 +244,5 @@
             </geometry>
         </collision>
-		<xacro:box_inertial mass="0.0001"
-                            x="0.001" y="0.001" z="0.001"
-                            pose_xyz = "0 0 0"
-                            pose_rpy = "0 0 0"/>
+		<xacro:small_inertial />
 		<contact>
 				<!--
@@ -273,8 +272,5 @@
 	</link>
     <link name="foot_link">
-		<xacro:box_inertial mass="0.0001"
-                            x="0.001" y="0.001" z="0.001"
-                            pose_xyz = "0 0 0"
-                            pose_rpy = "0 0 0"/>
+		<xacro:small_inertial />
 	</link>
 	<joint name="world_to_rail" type="fixed">
@@ -291,5 +287,5 @@
     <joint name="hip_joint" type="revolute">
     	<parent link="slider_link"/>
-    	<child link="thigh_link"/>
+    	<child link="thigh_link_base"/>
     	<origin xyz="0 ${hip_y_offset} 0" rpy="0 0 0"/>
 		<dynamics damping="0.0" friction="${hip_friction}"/>
@@ -297,11 +293,12 @@
         <axis xyz="0 1 0"/>
 	</joint>
-	<joint name="thigh_link_base" type="fixed">
-        <parent link="thigh_link"/>
-        <child link="thigh_link_base"/>
+	<joint name="thigh_link_com" type="fixed">
+        <parent link="thigh_link_base"/>
+        <child link="thigh_link_com"/>
+		<origin xyz="0 0 -${thigh_height/2}" rpy="0 0 0"/>
     </joint>
  	<joint name="knee_joint" type="revolute">
-    	<parent link="thigh_link"/>
-    	<child link="shin_link"/>
+    	<parent link="thigh_link_base"/>
+    	<child link="shin_link_base"/>
     	<origin xyz="0 ${knee_y_offset} -${thigh_height}" rpy="0 0 0"/>
 		<dynamics damping="0.0" friction="${knee_friction}"/>
@@ -309,15 +306,16 @@
         <axis xyz="0 1 0"/>
 	</joint>
-	<joint name="shin_link_base" type="fixed">
-        <parent link="shin_link"/>
-        <child link="shin_link_base"/>
+	<joint name="shin_link_com" type="fixed">
+        <parent link="shin_link_base"/>
+        <child link="shin_link_com"/>
+		<origin xyz="0 0 -${shin_height/2}" rpy="0 0 0"/>
     </joint>
 	<joint name="foot_center_joint" type="fixed">
-        <parent link="shin_link"/>
+        <parent link="shin_link_base"/>
         <child link="foot_center_link"/>
     	<origin xyz="0 0 -${shin_height-shin_width}" rpy="0 0 0"/>
     </joint>
 	<joint name="foot_joint" type="fixed">
-        <parent link="shin_link"/>
+        <parent link="shin_link_base"/>
         <child link="foot_link"/>
     	<origin xyz="0 0 -${shin_height}" rpy="0 0 0"/>

Commit message: Trying to figure out why xbot-gazebo has higher torques

File: src/jumping_leg/models/leg_simple.urdf.xacro (robot description, xacro)
@@ -140,5 +140,5 @@
 		<xacro:box_inertial mass="${slider_mass}"
                             x="${slider_width}" y="${slider_length}" z="${slider_height}"
-                            pose_xyz = "0 0 ${slider_height}"
+                            pose_xyz = "0 0 0"
                             pose_rpy = "0 0 0"/>
 	</link>
@@ -246,28 +246,28 @@
 		<xacro:small_inertial />
 		<contact>
-				<!--
-				Pybullet defaults maybe are these (from bullet3/examples/Importers/ImportURDFDemo/URDFJointTypes.h line 33)
-				URDFLinkContactInfo()
-					: m_lateralFriction(0.5),
-					m_rollingFriction(0),
-					m_spinningFriction(0),
-					m_restitution(0),
-					m_inertiaScaling(1),
-					m_contactCfm(0),
-					m_contactErp(0),
-					m_contactStiffness(1e4),
-					m_contactDamping(1)
-				-->
-				<lateral_friction value="0.9"/>
-				<rolling_friction value="0.01"/>
-				<!-- <contact_cfm value="0.1 "/> -->
-				<!-- <contact_erp value="0.2"/> -->
-				<restitution value="0.05"/>
-				<!-- <spinning_friction value="0"/> -->
-				<!-- <friction_anchor value="0"/> -->
-				<!-- <inertia_scaling value="0"/> -->
-				<!-- <stiffness value="2500"/>
-				<damping value="8"/>  -->
-			</contact>
+			<!--
+			Pybullet defaults maybe are these (from bullet3/examples/Importers/ImportURDFDemo/URDFJointTypes.h line 33)
+			URDFLinkContactInfo()
+				: m_lateralFriction(0.5),
+				m_rollingFriction(0),
+				m_spinningFriction(0),
+				m_restitution(0),
+				m_inertiaScaling(1),
+				m_contactCfm(0),
+				m_contactErp(0),
+				m_contactStiffness(1e4),
+				m_contactDamping(1)
+			-->
+			<lateral_friction value="0.9"/>
+			<rolling_friction value="0.01"/>
+			<!-- <contact_cfm value="0.1 "/> -->
+			<!-- <contact_erp value="0.2"/> -->
+			<restitution value="0.05"/>
+			<!-- <spinning_friction value="0"/> -->
+			<!-- <friction_anchor value="0"/> -->
+			<!-- <inertia_scaling value="0"/> -->
+			<!-- <stiffness value="2500"/>
+			<damping value="8"/>  -->
+		</contact>
 	</link>
     <link name="foot_link">
@@ -304,5 +304,5 @@
 		<dynamics damping="0.0" friction="${knee_friction}"/>
        	<limit lower="-2.4" upper="2.4" effort="112" velocity="20"/>
-        <axis xyz="0 1 0"/>
+        <axis xyz="0 -1 0"/>
 	</joint>
 	<joint name="shin_link_com" type="fixed">

File: src/jumping_leg/models/red_intangible_ball.urdf.xacro (robot description, xacro)
@@ -2,6 +2,8 @@
 <robot name="red_intangible_ball" xmlns:xacro="http://www.ros.org/wiki/xacro">
 	<xacro:arg name="radius" default="0.05" />
+	<xacro:arg name="add_world_link" default="False" />
 	<xacro:property name="radius" default="$(arg radius)" />
 	<xacro:property name="color_rgba" default="0.9 0.1 0.1 0.8" />
+	<xacro:property name="add_world_link" default="$(arg add_world_link)" />
 	<material name="red">
 		<color rgba="${color_rgba}"/>
@@ -21,5 +23,5 @@
                 <sphere radius="${radius}" />
             </geometry>
-			<material name="red"/>
+			<!-- <material name="red"/> -->
         </visual>
 		<xacro:box_inertial mass="0.001" x="${2*radius}" y="${2*radius}" z="${2*radius}" pose_xyz="0 0 0" pose_rpy="0 0 0"/>
@@ -28,12 +30,20 @@
 		<visual name="visual">
 			<material>
-			<ambient>"${color_rgba}"</ambient>
-			<diffuse>"${color_rgba}"</diffuse>
-			<!--
-			<specular>1 0 0 1</specular>
-			<emissive>1 0 0 1</emissive>
-			-->
+				<ambient>${color_rgba}</ambient>
+				<diffuse>${color_rgba}</diffuse>
+				<specular>0 0 0 1</specular>
+				<emissive>0 0 0 1</emissive>
 			</material>
       	</visual>
     </gazebo>
+	<gazebo>
+		<static>true</static>
+	</gazebo>
+	<xacro:if value="${add_world_link}">
+		<link name="world"/>
+		<joint name="world_joint" type="fixed">
+			<parent link="world"/>
+			<child link="sphere_link"/>
+		</joint>
+	</xacro:if>
 </robot>

File: src/jumping_leg/models/support.urdf.xacro (robot description, xacro)
@@ -4,8 +4,10 @@
 	<xacro:arg name="size_y" default="0.50" />
 	<xacro:arg name="size_z" default="0.005" />
+	<xacro:arg name="add_world_link" default="True" />
 	<xacro:property name="size_x" default="$(arg size_x)" />
 	<xacro:property name="size_y" default="$(arg size_y)" />
 	<xacro:property name="size_z" default="$(arg size_z)" />
 	<xacro:property name="color_rgba" default="0.3 0.3 0.3 1.0" />
+	<xacro:property name="add_world_link" default="$(arg add_world_link)" />
 	<material name="support_color">
 		<color rgba="${color_rgba}"/>
@@ -18,5 +20,4 @@
 		</inertial>
 	</xacro:macro>
-    <!-- <link name="world"/> -->
 	<link name="plate">
 		<!-- The shin is made of a cylinder plus a sphere, the total length, is shin_height, so the length  of the two are detemrined accordingly -->
@@ -73,3 +74,13 @@
       	</visual>
     </gazebo>
+	<gazebo>
+		<static>true</static>
+	</gazebo>
+	<xacro:if value="${add_world_link}">
+		<link name="world"/>
+		<joint name="world_joint" type="fixed">
+			<parent link="world"/>
+			<child link="plate"/>
+		</joint>
+	</xacro:if>
 </robot>
