Commit message: LocomotionEnv, lower dampings

File: src/jumping_leg/models/quad_simple.urdf.xacro (robot description, xacro)
@@ -2,5 +2,5 @@
 <robot name="quad_simple" xmlns:xacro="http://www.ros.org/wiki/xacro">
     <xacro:include filename="package://jumping_leg/models/commons.xacro"/>
-    <xacro:include filename="package://jumping_leg/models/leg_simple.xacro"/>
+    <xacro:include filename="$(find jumping_leg)/models/leg_simple.xacro"/>
 	<!-- <xacro:arg name="hip_out_offset" default="0.2146" />  -->
 	<xacro:arg name="hip_out_offset" default="0.05" />
@@ -40,5 +40,4 @@
 	<xacro:property name="knee_friction" default="$(arg knee_friction)" />
 	<xacro:property name="hip_friction" default="$(arg hip_friction)" />
-    <link name="world"/>
     <link name="body_link">
 		<visual name = "body_link_v">
@@ -123,7 +122,8 @@
                         parent_link = "body_link"
                         leg_name = "back_right"/>
+    <!-- <link name="world"/>
 	<joint name="world_to_body" type="floating">
         <parent link="world"/>
         <child link="body_link"/>
-    </joint>
+    </joint> -->
 </robot>

Commit message: sac_cheetah works kinda nice, going back to quad

File: src/jumping_leg/models/quad_simple.urdf.xacro (robot description, xacro)
@@ -43,6 +43,6 @@
 	<xacro:property name="knee_friction" default="$(arg knee_friction)" />
 	<xacro:property name="hip_friction" default="$(arg hip_friction)" />
-    <xacro:property name="hip_x_min_pos" default="0.0" />
-    <xacro:property name="hip_x_max_pos" default="2.4" />
+    <xacro:property name="hip_x_min_pos" default="-2.4" />
+    <xacro:property name="hip_x_max_pos" default="0.0" />
     <xacro:property name="hip_y_min_pos" default="-2.4" />
     <xacro:property name="hip_y_max_pos" default="2.4" />

Commit message: jpose randomization

File: src/jumping_leg/models/quad_simple.urdf.xacro (robot description, xacro)
@@ -183,8 +183,8 @@
                         knee_max_pos = "${knee_max_pos}"
                         />
-    <!-- <link name="world"/>
+    <link name="world"/>
 	<joint name="world_to_body" type="floating">
         <parent link="world"/>
         <child link="body_link"/>
-    </joint> -->
+    </joint>
 </robot>
