Commit message: Fixed quadruped initial pose

File: src/jumping_leg/models/leg_simple.xacro (robot description, xacro)
@@ -16,5 +16,12 @@
 											knee_friction
 											parent_link
-											leg_name">
+											leg_name
+											is_left_leg:=true">
+			<xacro:if value="${is_left_leg}">
+				<xacro:property name="exterior_y_direction" value="1"/>
+			</xacro:if>
+			<xacro:unless value="${is_left_leg}">
+				<xacro:property name="exterior_y_direction" value="-1"/>
+			</xacro:unless>
 			<link name="prethigh_link_${leg_name}">
 				<xacro:small_inertial/>
@@ -128,13 +135,13 @@
 				<xacro:small_inertial />
 			</link>
-			<joint name="hip_joint1_${leg_name}" type="revolute">
+			<joint name="hip_joint_y_${leg_name}" type="revolute">
 				<parent link="${parent_link}"/>
 				<child link="prethigh_link_${leg_name}"/>
-				<origin xyz="${hip_x_offset} ${hip_y_offset} ${hip_z_offset}" rpy="0 0 0"/>
+				<origin xyz="${hip_x_offset} ${exterior_y_direction*hip_y_offset} ${hip_z_offset}" rpy="0 0 0"/>
 				<dynamics damping="0.0" friction="${hip_friction}"/>
 				<limit lower="-2.4" upper="2.4" effort="112" velocity="20"/>
 				<axis xyz="0 1 0"/>
 			</joint>
-			<joint name="hip_joint2_${leg_name}" type="revolute">
+			<joint name="hip_joint_x_${leg_name}" type="revolute">
 				<parent link="prethigh_link_${leg_name}"/>
 				<child link="thigh_link_${leg_name}"/>
@@ -142,5 +149,5 @@
 				<dynamics damping="0.0" friction="${hip_friction}"/>
 				<limit lower="-2.4" upper="2.4" effort="112" velocity="20"/>
-				<axis xyz="1 0 0"/>
+				<axis xyz="${exterior_y_direction} 0 0"/>
 			</joint>
 			<joint name="thigh_link_com_${leg_name}" type="fixed">
@@ -152,5 +159,5 @@
 				<parent link="thigh_link_${leg_name}"/>
 				<child link="shin_link_${leg_name}"/>
-				<origin xyz="0 ${knee_y_offset} -${thigh_height}" rpy="0 0 0"/>
+				<origin xyz="0 ${exterior_y_direction*knee_y_offset} -${thigh_height}" rpy="0 0 0"/>
 				<dynamics damping="0.0" friction="${knee_friction}"/>
 				<limit lower="-2.4" upper="2.4" effort="112" velocity="20"/>

File: src/jumping_leg/models/quad_simple.urdf.xacro (robot description, xacro)
@@ -73,7 +73,8 @@
                         knee_friction = "${knee_friction}"
                         parent_link = "body_link"
-                        leg_name = "front_left"/>
+                        leg_name = "front_left"
+                        is_left_leg = "true"/>
     <xacro:leg_simple   hip_x_offset = "${front_legs_pos}"
-                        hip_y_offset = "${-body_width/2 - legs_out_offset}"
+                        hip_y_offset = "${body_width/2 + legs_out_offset}"
                         hip_z_offset = "0"
                         thigh_width  = "${thigh_width}"
@@ -81,5 +82,5 @@
                         thigh_mass = "${thigh_mass}"
                         thigh_color = "${thigh_color}"
-                        knee_y_offset = "${-knee_y_offset}"
+                        knee_y_offset = "${knee_y_offset}"
                         shin_width = "${shin_width}"
                         shin_height = "${shin_height}"
@@ -89,5 +90,6 @@
                         knee_friction = "${knee_friction}"
                         parent_link = "body_link"
-                        leg_name = "front_right"/>
+                        leg_name = "front_right"
+                        is_left_leg = "false"/>
     <xacro:leg_simple   hip_x_offset = "${back_legs_pos}"
                         hip_y_offset = "${body_width/2 + legs_out_offset}"
@@ -105,7 +107,8 @@
                         knee_friction = "${knee_friction}"
                         parent_link = "body_link"
-                        leg_name = "back_left"/>
+                        leg_name = "back_left"
+                        is_left_leg = "true"/>
     <xacro:leg_simple   hip_x_offset = "${back_legs_pos}"
-                        hip_y_offset = "${-body_width/2 - legs_out_offset}"
+                        hip_y_offset = "${body_width/2 + legs_out_offset}"
                         hip_z_offset = "0"
                         thigh_width  = "${thigh_width}"
@@ -113,5 +116,5 @@
                         thigh_mass = "${thigh_mass}"
                         thigh_color = "${thigh_color}"
-                        knee_y_offset = "${-knee_y_offset}"
+                        knee_y_offset = "${knee_y_offset}"
                         shin_width = "${shin_width}"
                         shin_height = "${shin_height}"
@@ -121,5 +124,6 @@
                         knee_friction = "${knee_friction}"
                         parent_link = "body_link"
-                        leg_name = "back_right"/>
+                        leg_name = "back_right"
+                        is_left_leg = "false"/>
     <!-- <link name="world"/>
 	<joint name="world_to_body" type="floating">

Commit message: changing hip orientation, introducing control ranges

File: src/jumping_leg/models/leg_simple.xacro (robot description, xacro)
@@ -146,5 +146,5 @@
 				<parent link="prethigh_link_${leg_name}"/>
 				<child link="thigh_link_${leg_name}"/>
-				<origin xyz="0 0 0" rpy="0 0 0"/>
+				<origin xyz="0 0 0" rpy="${exterior_y_direction*3.14159/2} 0 0"/>
 				<dynamics damping="0.0" friction="${hip_friction}"/>
 				<limit lower="-2.4" upper="2.4" effort="112" velocity="20"/>

Commit message: improvements locomotion env

File: src/jumping_leg/models/leg_simple.xacro (robot description, xacro)
@@ -1,4 +1,23 @@
 <?xml version="1.0" encoding="utf-8"  ?>
 <robot xmlns:xacro="http://www.ros.org/wiki/xacro">
+    <xacro:macro name="leg_contact_params" params="">
+        <contact>
+        <!--
+        Defaults maybe are these (from bullet3/examples/Importers/ImportURDFDemo/URDFJointTypes.h line 33)
+        URDFLinkContactInfo()
+            : m_lateralFriction(0.5),
+            m_rollingFriction(0),
+            m_spinningFriction(0),
+            m_restitution(0),
+            m_inertiaScaling(1),
+            m_contactCfm(0),
+            m_contactErp(0),
+            m_contactStiffness(1e4),
+            m_contactDamping(1)
+        -->
+            <lateral_friction value="1"/>
+            <rolling_friction value="0.00001"/>
+        </contact>
+    </xacro:macro>
 	<xacro:macro name="leg_simple" params="hip_x_offset
 											hip_y_offset
@@ -41,4 +60,5 @@
 				</collision>
 				<xacro:small_inertial />
+		        <xacro:leg_contact_params />
 			</link>
 			<link name="thigh_link_com_${leg_name}">
@@ -74,4 +94,5 @@
 				</collision>
 				<xacro:small_inertial />
+		        <xacro:leg_contact_params />
 			</link>
 			<link name="shin_link_com_${leg_name}">
@@ -86,9 +107,4 @@
 					</material>
 				</visual>
-				<contact>
-					<lateral_friction value="0.01"/>
-					<rolling_friction value="0.01"/>
-					<restitution value="0.05"/>
-				</contact>
 			</gazebo>
 			<link name="foot_center_link_${leg_name}">

File: src/jumping_leg/models/quad_simple.urdf.xacro (robot description, xacro)
@@ -40,4 +40,23 @@
 	<xacro:property name="knee_friction" default="$(arg knee_friction)" />
 	<xacro:property name="hip_friction" default="$(arg hip_friction)" />
+    <xacro:macro name="default_contact_params" params="">
+        <contact>
+        <!--
+        Defaults maybe are these (from bullet3/examples/Importers/ImportURDFDemo/URDFJointTypes.h line 33)
+        URDFLinkContactInfo()
+            : m_lateralFriction(0.5),
+            m_rollingFriction(0),
+            m_spinningFriction(0),
+            m_restitution(0),
+            m_inertiaScaling(1),
+            m_contactCfm(0),
+            m_contactErp(0),
+            m_contactStiffness(1e4),
+            m_contactDamping(1)
+        -->
+            <lateral_friction value="1"/>
+            <rolling_friction value="0.00001"/>
+        </contact>
+    </xacro:macro>
     <link name="body_link">
 		<visual name = "body_link_v">
@@ -57,4 +76,5 @@
                             pose_xyz = "0 0 0"
                             pose_rpy = "0 0 0"/>
+        <xacro:default_contact_params />
 	</link>
     <xacro:leg_simple   hip_x_offset = "${front_legs_pos}"

Commit message: some improvements

File: src/jumping_leg/models/leg_simple.xacro (robot description, xacro)
@@ -36,5 +36,11 @@
 											parent_link
 											leg_name
-											is_left_leg:=true">
+											is_left_leg:=true
+											hip_x_min_pos:=-2.4
+											hip_x_max_pos:=2.4
+											hip_y_min_pos:=-2.4
+											hip_y_max_pos:=2.4
+											knee_min_pos:=-2.4
+											knee_max_pos:=2.4">
 			<xacro:if value="${is_left_leg}">
 				<xacro:property name="exterior_y_direction" value="1"/>

File: src/jumping_leg/models/quad_simple.urdf.xacro (robot description, xacro)
@@ -43,4 +43,10 @@
 	<xacro:property name="knee_friction" default="$(arg knee_friction)" />
 	<xacro:property name="hip_friction" default="$(arg hip_friction)" />
+    <xacro:property name="hip_x_min_pos" default="0.0" />
+    <xacro:property name="hip_x_max_pos" default="2.4" />
+    <xacro:property name="hip_y_min_pos" default="-2.4" />
+    <xacro:property name="hip_y_max_pos" default="2.4" />
+    <xacro:property name="knee_min_pos" default="-2.4" />
+    <xacro:property name="knee_max_pos" default="2.4" />
     <xacro:macro name="default_contact_params" params="">
         <contact>
@@ -97,5 +103,12 @@
                         parent_link = "body_link"
                         leg_name = "front_left"
-                        is_left_leg = "true"/>
+                        is_left_leg = "true"
+                        hip_x_min_pos = "${hip_x_min_pos}"
+                        hip_x_max_pos = "${hip_x_max_pos}"
+                        hip_y_min_pos = "${hip_y_min_pos}"
+                        hip_y_max_pos = "${hip_y_max_pos}"
+                        knee_min_pos = "${knee_min_pos}"
+                        knee_max_pos = "${knee_max_pos}"
+                        />
     <xacro:leg_simple   hip_x_offset = "${front_legs_pos}"
                         hip_y_offset = "${body_width/2 + legs_out_offset}"
@@ -114,5 +127,12 @@
                         parent_link = "body_link"
                         leg_name = "front_right"
-                        is_left_leg = "false"/>
+                        is_left_leg = "false"
+                        hip_x_min_pos = "${hip_x_min_pos}"
+                        hip_x_max_pos = "${hip_x_max_pos}"
+                        hip_y_min_pos = "${hip_y_min_pos}"
+                        hip_y_max_pos = "${hip_y_max_pos}"
+                        knee_min_pos = "${knee_min_pos}"
+                        knee_max_pos = "${knee_max_pos}"
+                        />
     <xacro:leg_simple   hip_x_offset = "${back_legs_pos}"
                         hip_y_offset = "${body_width/2 + legs_out_offset}"
@@ -131,5 +151,12 @@
                         parent_link = "body_link"
                         leg_name = "back_left"
-                        is_left_leg = "true"/>
+                        is_left_leg = "true"
+                        hip_x_min_pos = "${hip_x_min_pos}"
+                        hip_x_max_pos = "${hip_x_max_pos}"
+                        hip_y_min_pos = "${hip_y_min_pos}"
+                        hip_y_max_pos = "${hip_y_max_pos}"
+                        knee_min_pos = "${knee_min_pos}"
+                        knee_max_pos = "${knee_max_pos}"
+                        />
     <xacro:leg_simple   hip_x_offset = "${back_legs_pos}"
                         hip_y_offset = "${body_width/2 + legs_out_offset}"
@@ -148,5 +175,12 @@
                         parent_link = "body_link"
                         leg_name = "back_right"
-                        is_left_leg = "false"/>
+                        is_left_leg = "false"
+                        hip_x_min_pos = "${hip_x_min_pos}"
+                        hip_x_max_pos = "${hip_x_max_pos}"
+                        hip_y_min_pos = "${hip_y_min_pos}"
+                        hip_y_max_pos = "${hip_y_max_pos}"
+                        knee_min_pos = "${knee_min_pos}"
+                        knee_max_pos = "${knee_max_pos}"
+                        />
     <!-- <link name="world"/>
 	<joint name="world_to_body" type="floating">

Commit message: almost there

File: src/jumping_leg/models/leg_simple.xacro (robot description, xacro)
@@ -19,4 +19,18 @@
             <rolling_friction value="0.00001"/>
         </contact>
+    </xacro:macro>
+	<xacro:macro name="bar" params="use_cylinder
+									length
+									thickness">
+        <xacro:if value="${use_cylinder}">
+			<geometry>
+				<cylinder length="${length}" radius="${thickness/2}" />
+			</geometry>
+		</xacro:if>
+		<xacro:unless value="${use_cylinder}">
+			<geometry>
+				<box size="${thickness} ${thickness} ${length}" />
+			</geometry>
+		</xacro:unless>
     </xacro:macro>
 	<xacro:macro name="leg_simple" params="hip_x_offset
@@ -42,5 +56,6 @@
 											hip_y_max_pos:=2.4
 											knee_min_pos:=-2.4
-											knee_max_pos:=2.4">
+											knee_max_pos:=2.4
+											use_cylinders:=true">
 			<xacro:if value="${is_left_leg}">
 				<xacro:property name="exterior_y_direction" value="1"/>
@@ -55,13 +70,9 @@
 				<visual name = "thigh_link_v_${leg_name}">
 					<origin xyz="0 0 -${thigh_height/2}" rpy="0 0 0"/>
-					<geometry>
-						<cylinder length="${thigh_height}" radius="${thigh_width/2}" />
-					</geometry>
+					<xacro:bar length="${thigh_height}" thickness="${thigh_width}" use_cylinder="${use_cylinders}"/>
 				</visual>
 				<collision name = "thigh_link_c_${leg_name}">
 					<origin xyz="0 0 -${thigh_height/2}" rpy="0 0 0"/>
-					<geometry>
-						<cylinder length="${thigh_height}" radius="${thigh_width/2}" />
-					</geometry>
+					<xacro:bar length="${thigh_height}" thickness="${thigh_width}" use_cylinder="${use_cylinders}"/>
 				</collision>
 				<xacro:small_inertial />
@@ -89,13 +100,9 @@
 				<visual name = "shin_link_v_${leg_name}">
 					<origin xyz="0 0 -${(shin_height-shin_width)/2}" rpy="0 0 0"/>
-					<geometry>
-						<cylinder length="${shin_height-shin_width}" radius="${shin_width/2}" />
-					</geometry>
+					<xacro:bar length="${shin_height-shin_width}" thickness="${shin_width}" use_cylinder="${use_cylinders}"/>
 				</visual>
 				<collision name = "shin_link_c_${leg_name}">
 					<origin xyz="0 0 -${(shin_height-shin_width)/2}" rpy="0 0 0"/>
-					<geometry>
-						<cylinder length="${shin_height-shin_width}" radius="${shin_width/2}" />
-					</geometry>
+					<xacro:bar length="${shin_height-shin_width}" thickness="${shin_width}" use_cylinder="${use_cylinders}"/>
 				</collision>
 				<xacro:small_inertial />

File: src/jumping_leg/models/quad_simple.urdf.xacro (robot description, xacro)
@@ -25,4 +25,5 @@
 	<xacro:arg name="hip_friction" default="0.1" />
 	<xacro:arg name="knee_friction" default="0.1" />
+	<xacro:arg name="use_cylinders" default="True" />
 	<xacro:property name="legs_out_offset"  default="$(arg hip_out_offset)" />
 	<xacro:property name="front_legs_pos"  default="$(arg front_legs_pos)" />
@@ -43,4 +44,5 @@
 	<xacro:property name="knee_friction" default="$(arg knee_friction)" />
 	<xacro:property name="hip_friction" default="$(arg hip_friction)" />
+	<xacro:property name="use_cylinders" default="$(arg use_cylinders)" />
     <xacro:property name="hip_x_min_pos" default="-2.4" />
     <xacro:property name="hip_x_max_pos" default="0.0" />
@@ -110,4 +112,5 @@
                         knee_min_pos = "${knee_min_pos}"
                         knee_max_pos = "${knee_max_pos}"
+                        use_cylinders = "${use_cylinders}"
                         />
     <xacro:leg_simple   hip_x_offset = "${front_legs_pos}"
@@ -134,4 +137,5 @@
                         knee_min_pos = "${knee_min_pos}"
                         knee_max_pos = "${knee_max_pos}"
+                        use_cylinders = "${use_cylinders}"
                         />
     <xacro:leg_simple   hip_x_offset = "${back_legs_pos}"
@@ -158,4 +162,5 @@
                         knee_min_pos = "${knee_min_pos}"
                         knee_max_pos = "${knee_max_pos}"
+                        use_cylinders = "${use_cylinders}"
                         />
     <xacro:leg_simple   hip_x_offset = "${back_legs_pos}"
@@ -182,4 +187,5 @@
                         knee_min_pos = "${knee_min_pos}"
                         knee_max_pos = "${knee_max_pos}"
+                        use_cylinders = "${use_cylinders}"
                         />
     <link name="world"/>

Commit message: improvements

File: src/jumping_leg/models/leg_simple.xacro (robot description, xacro)
@@ -71,4 +71,7 @@
 					<origin xyz="0 0 -${thigh_height/2}" rpy="0 0 0"/>
 					<xacro:bar length="${thigh_height}" thickness="${thigh_width}" use_cylinder="${use_cylinders}"/>
+					<material name="DarkOrange">
+						<color rgba="0.95 0.50 0.1 1.0"/>
+					</material>
 				</visual>
 				<collision name = "thigh_link_c_${leg_name}">
@@ -101,4 +104,7 @@
 					<origin xyz="0 0 -${(shin_height-shin_width)/2}" rpy="0 0 0"/>
 					<xacro:bar length="${shin_height-shin_width}" thickness="${shin_width}" use_cylinder="${use_cylinders}"/>
+					<material name="orange">
+						<color rgba="0.95 0.60 0.1 1.0"/>
+					</material>
 				</visual>
 				<collision name = "shin_link_c_${leg_name}">
@@ -127,4 +133,7 @@
 						<sphere radius="${shin_width}" />
 					</geometry>
+					<material name="grey">
+						<color rgba="0.3 0.2 0.1 1.0"/>
+					</material>
 				</visual>
 				<collision>

File: src/jumping_leg/models/quad_simple.urdf.xacro (robot description, xacro)
@@ -76,4 +76,7 @@
 				<box size="${body_length} ${body_width} ${body_height}"/>
 			</geometry>
+            <material name="light_orange">
+                <color rgba="0.85 0.30 0.1 1.0"/>
+            </material>
 	   	</visual>
   		<collision name = "body_link_c">

File: src/jumping_leg/models/red_arrow.urdf.xacro (robot description, xacro)
@@ -1,4 +1,4 @@
 <?xml version="1.0" encoding="utf-8"  ?>
-<robot name="red_intangible_ball" xmlns:xacro="http://www.ros.org/wiki/xacro">
+<robot name="arrow" xmlns:xacro="http://www.ros.org/wiki/xacro">
 	<xacro:arg name="add_world_link" default="False" />
 	<xacro:property name="color_rgba" default="0.9 0.1 0.1 0.8" />
