Commit message: many fixes

File: src/jumping_leg/models/axes.urdf.xacro (robot description, xacro)
@@ -5,11 +5,11 @@
 	<xacro:property name="add_world_link" default="$(arg add_world_link)" />
 	<material name="red">
-		<color rgba="1 0 0 0.8"/>
+		<color rgba="1 0 0 0.6"/>
 	</material>
 	<material name="green">
-		<color rgba="0 1 0 0.8"/>
+		<color rgba="0 1 0 0.6"/>
 	</material>
 	<material name="blue">
-		<color rgba="0 0 1 0.8"/>
+		<color rgba="0 0 1 0.6"/>
 	</material>
 	<xacro:macro name="box_inertial" params="mass x y z pose_xyz pose_rpy">

File: src/jumping_leg/models/cheetah.urdf.xacro (robot description, xacro)
@@ -37,6 +37,4 @@
 	<xacro:property name="knee_friction" default="$(arg knee_friction)" />
 	<xacro:property name="hip_friction" default="$(arg hip_friction)" />
-    <xacro:property name="hip_x_min_pos" default="0.0" />
-    <xacro:property name="hip_x_max_pos" default="2.4" />
     <xacro:property name="hip_y_min_pos" default="-2.4" />
     <xacro:property name="hip_y_max_pos" default="2.4" />
@@ -63,4 +61,6 @@
     </xacro:macro>
     <link name="world"/>
+    <link name="mid"/>
+    <link name="mid2"/>
     <link name="body_link">
 		<visual name = "body_link_v">
@@ -90,5 +90,5 @@
     </joint>
     <joint name="torso_z_slider" type="prismatic">
-        <origin xyz="0 0 1.0" rpy="0 0 0" />
+        <origin xyz="0 0 0" rpy="0 0 0" />
         <axis xyz="0 0 1" rpy="0 0 0" />
         <parent link="mid"/>

Commit message: MJX efficiency improvements, fixed vec-based pybullet pipeline

File: src/jumping_leg/models/axes.urdf.xacro (robot description, xacro)
@@ -1,4 +1,4 @@
 <?xml version="1.0" encoding="utf-8"  ?>
-<robot name="red_intangible_ball" xmlns:xacro="http://www.ros.org/wiki/xacro">
+<robot name="axes" xmlns:xacro="http://www.ros.org/wiki/xacro">
 	<xacro:arg name="add_world_link" default="False" />
 	<xacro:property name="color_rgba" default="0.9 0.1 0.1 0.8" />

File: src/jumping_leg/models/leg_simple.xacro (robot description, xacro)
@@ -57,5 +57,7 @@
 											knee_min_pos:=-2.4
 											knee_max_pos:=2.4
-											use_cylinders:=true">
+											use_cylinders:=true
+											enable_thigh_collisions:=true
+											enable_shin_collisions:=true">
 			<xacro:if value="${is_left_leg}">
 				<xacro:property name="exterior_y_direction" value="1"/>
@@ -75,8 +77,10 @@
 					</material>
 				</visual>
-				<collision name = "thigh_link_c_${leg_name}">
-					<origin xyz="0 0 -${thigh_height/2}" rpy="0 0 0"/>
-					<xacro:bar length="${thigh_height}" thickness="${thigh_width}" use_cylinder="${use_cylinders}"/>
-				</collision>
+        		<xacro:if value="${enable_thigh_collisions}">
+					<collision name = "thigh_link_c_${leg_name}">
+						<origin xyz="0 0 -${thigh_height/2}" rpy="0 0 0"/>
+						<xacro:bar length="${thigh_height}" thickness="${thigh_width}" use_cylinder="${use_cylinders}"/>
+					</collision>
+				</xacro:if>
 				<xacro:small_inertial />
 		        <xacro:leg_contact_params />
@@ -108,8 +112,10 @@
 					</material>
 				</visual>
-				<collision name = "shin_link_c_${leg_name}">
-					<origin xyz="0 0 -${(shin_height-shin_width)/2}" rpy="0 0 0"/>
-					<xacro:bar length="${shin_height-shin_width}" thickness="${shin_width}" use_cylinder="${use_cylinders}"/>
-				</collision>
+        		<xacro:if value="${enable_shin_collisions}">
+					<collision name = "shin_link_c_${leg_name}">
+						<origin xyz="0 0 -${(shin_height-shin_width)/2}" rpy="0 0 0"/>
+						<xacro:bar length="${shin_height-shin_width}" thickness="${shin_width}" use_cylinder="${use_cylinders}"/>
+					</collision>
+				</xacro:if>
 				<xacro:small_inertial />
 		        <xacro:leg_contact_params />

File: src/jumping_leg/models/quad_simple.urdf.xacro (robot description, xacro)
@@ -45,4 +45,10 @@
 	<xacro:property name="hip_friction" default="$(arg hip_friction)" />
 	<xacro:property name="use_cylinders" default="$(arg use_cylinders)" />
+	<xacro:arg name="enable_body_collisions" default="False" />
+	<xacro:arg name="enable_thigh_collisions" default="False" />
+	<xacro:arg name="enable_shin_collisions" default="False" />
+	<xacro:property name="enable_body_collisions" default="$(arg enable_body_collisions)" />
+	<xacro:property name="enable_thigh_collisions" default="$(arg enable_thigh_collisions)" />
+	<xacro:property name="enable_shin_collisions" default="$(arg enable_shin_collisions)" />
     <xacro:property name="hip_x_min_pos" default="-2.4" />
     <xacro:property name="hip_x_max_pos" default="0.0" />
@@ -80,10 +86,12 @@
             </material>
 	   	</visual>
-  		<collision name = "body_link_c">
-			<origin xyz="0 0 0" rpy="0 0 0"/>
-			<geometry>
-				<box size="${body_length} ${body_width} ${body_height}"/>
-			</geometry>
-	   	</collision>
+        <xacro:if value="${enable_body_collisions}">
+            <collision name = "body_link_c">
+                <origin xyz="0 0 0" rpy="0 0 0"/>
+                <geometry>
+                    <box size="${body_length} ${body_width} ${body_height}"/>
+                </geometry>
+            </collision>
+		</xacro:if>
 		<xacro:box_inertial mass="${body_mass}"
                             x="${body_width}" y="${body_length}" z="${body_height}"
@@ -116,4 +124,6 @@
                         knee_max_pos = "${knee_max_pos}"
                         use_cylinders = "${use_cylinders}"
+                        enable_thigh_collisions = "${enable_thigh_collisions}"
+                        enable_shin_collisions = "${enable_shin_collisions}"
                         />
     <xacro:leg_simple   hip_x_offset = "${front_legs_pos}"
@@ -141,4 +151,6 @@
                         knee_max_pos = "${knee_max_pos}"
                         use_cylinders = "${use_cylinders}"
+                        enable_thigh_collisions = "${enable_thigh_collisions}"
+                        enable_shin_collisions = "${enable_shin_collisions}"
                         />
     <xacro:leg_simple   hip_x_offset = "${back_legs_pos}"
@@ -166,4 +178,6 @@
                         knee_max_pos = "${knee_max_pos}"
                         use_cylinders = "${use_cylinders}"
+                        enable_thigh_collisions = "${enable_thigh_collisions}"
+                        enable_shin_collisions = "${enable_shin_collisions}"
                         />
     <xacro:leg_simple   hip_x_offset = "${back_legs_pos}"
@@ -191,4 +205,6 @@
                         knee_max_pos = "${knee_max_pos}"
                         use_cylinders = "${use_cylinders}"
+                        enable_thigh_collisions = "${enable_thigh_collisions}"
+                        enable_shin_collisions = "${enable_shin_collisions}"
                         />
     <link name="world"/>

Commit message: fix com body state usage, removed some mesh usage, automatically disable discard visuals

File: src/jumping_leg/models/axes.urdf.xacro (robot description, xacro)
@@ -22,7 +22,8 @@
 	<link name="x_arrow">
         <visual>
-			<origin xyz="0.1 0 0" rpy="0 0 0"/>
+			<origin xyz="0.5 0 0" rpy="0 0 0"/>
             <geometry>
-                <mesh filename="package://jumping_leg/models/arrow.stl"  scale="0.001 0.001 0.001"/>
+				<box size="1 0.1 0.1"/>
+                <!-- <mesh filename="package://jumping_leg/models/arrow.stl"  scale="0.001 0.001 0.001"/> -->
             </geometry>
 			<material name="red"/>
@@ -42,7 +43,8 @@
 	<link name="y_arrow">
         <visual>
-			<origin xyz="0 0.1 0" rpy="0 0 1.5707"/>
+			<origin xyz="0 0.5 0" rpy="0 0 1.5707"/>
             <geometry>
-                <mesh filename="package://jumping_leg/models/arrow.stl"  scale="0.001 0.001 0.001"/>
+				<box size="1 0.1 0.1"/>
+                <!-- <mesh filename="package://jumping_leg/models/arrow.stl"  scale="0.001 0.001 0.001"/> -->
             </geometry>
 			<material name="green"/>
@@ -62,7 +64,8 @@
 	<link name="z_arrow">
         <visual>
-			<origin xyz="0 0 0.1" rpy="0 -1.5707 0"/>
+			<origin xyz="0 0 0.5" rpy="0 -1.5707 0"/>
             <geometry>
-                <mesh filename="package://jumping_leg/models/arrow.stl"  scale="0.001 0.001 0.001"/>
+				<box size="1 0.1 0.1"/>
+                <!-- <mesh filename="package://jumping_leg/models/arrow.stl"  scale="0.001 0.001 0.001"/> -->
             </geometry>
 			<material name="blue"/>

File: src/jumping_leg/models/commons.xacro (robot description, xacro)
@@ -5,5 +5,7 @@
 			<origin xyz="${pose_xyz}" rpy="${pose_rpy}"/>
 			<mass value="${mass}" />
-			<inertia ixx="${0.083 * mass * (y*y + z*z)}" ixy="0.0" ixz="0.0" iyy="${0.083 * mass * (x*x + z*z)}" iyz="0.0" izz="${0.083 * mass * (x*x + y*y)}"/>
+			<inertia 	ixx="${0.083 * mass * (y*y + z*z)}" ixy="0.0" ixz="0.0"
+						iyy="${0.083 * mass * (x*x + z*z)}" iyz="0.0"
+						izz="${0.083 * mass * (x*x + y*y)}"/>
 		</inertial>
 	</xacro:macro>

File: src/jumping_leg/models/quad_simple.urdf.xacro (robot description, xacro)
@@ -96,5 +96,5 @@
 		</xacro:if>
 		<xacro:box_inertial mass="${body_mass}"
-                            x="${body_width}" y="${body_length}" z="${body_height}"
+                            x="${body_length}" y="${body_width}" z="${body_height}"
                             pose_xyz = "0 0 0"
                             pose_rpy = "0 0 0"/>
@@ -214,6 +214,6 @@
         <child link="body_link"/>
     </joint>
-  <mujoco>
+  <!-- <mujoco>
     <compiler  discardvisual="false"/>
-  </mujoco>
+  </mujoco> -->
 </robot>

File: src/jumping_leg/models/red_arrow.urdf.xacro (robot description, xacro)
@@ -17,7 +17,8 @@
 		<!-- The shin is made of a cylinder plus a sphere, the total length, is shin_height, so the length  of the two are detemrined accordingly -->
         <visual>
-			<origin xyz="0 0 0" rpy="0 0 0"/>
+			<origin xyz="0.5 0 0" rpy="0 0 0"/>
             <geometry>
-                <mesh filename="package://jumping_leg/models/arrow.stl"  scale="0.001 0.001 0.001"/>
+				<box size="1 0.1 0.1"/>
+                <!-- <mesh filename="package://jumping_leg/models/arrow.stl"  scale="0.001 0.001 0.001"/> -->
             </geometry>
 			<material name="red"/>
