Commit message: working on graspenv

File: src/adarl_envs/models/axes.urdf.xacro (robot description, xacro)
@@ -2,6 +2,8 @@
 <robot name="axes" xmlns:xacro="http://www.ros.org/wiki/xacro">
 	<xacro:arg name="add_world_link" default="False" />
+	<xacro:arg name="size" default="1.0" />
 	<xacro:property name="color_rgba" default="0.9 0.1 0.1 0.8" />
 	<xacro:property name="add_world_link" default="$(arg add_world_link)" />
+	<xacro:property name="size" default="$(arg size)" />
 	<material name="red">
 		<color rgba="1 0 0 0.6"/>
@@ -22,7 +24,7 @@
 	<link name="x_arrow">
         <visual>
-			<origin xyz="0.5 0 0" rpy="0 0 0"/>
+			<origin xyz="${size/2} 0 0" rpy="0 0 0"/>
             <geometry>
-				<box size="1 0.1 0.1"/>
+				<box size="${size} ${0.1*size} ${0.1*size}"/>
                 <!-- <mesh filename="package://adarl_envs/models/arrow.stl"  scale="0.001 0.001 0.001"/> -->
             </geometry>
@@ -43,7 +45,7 @@
 	<link name="y_arrow">
         <visual>
-			<origin xyz="0 0.5 0" rpy="0 0 1.5707"/>
+			<origin xyz="0 ${size/2} 0" rpy="0 0 1.5707"/>
             <geometry>
-				<box size="1 0.1 0.1"/>
+				<box size="${size} ${0.1*size} ${0.1*size}"/>
                 <!-- <mesh filename="package://adarl_envs/models/arrow.stl"  scale="0.001 0.001 0.001"/> -->
             </geometry>
@@ -64,7 +66,7 @@
 	<link name="z_arrow">
         <visual>
-			<origin xyz="0 0 0.5" rpy="0 -1.5707 0"/>
+			<origin xyz="0 0 ${size/2}" rpy="0 -1.5707 0"/>
             <geometry>
-				<box size="1 0.1 0.1"/>
+				<box size="${size} ${0.1*size} ${0.1*size}"/>
                 <!-- <mesh filename="package://adarl_envs/models/arrow.stl"  scale="0.001 0.001 0.001"/> -->
             </geometry>
