Commit message: Changed a bit actacc, ground time reward, pitchnroll velocity & error velocity , heading kd

File: src/adarl_envs/models/red_arrow.urdf.xacro (robot description, xacro)
@@ -2,8 +2,9 @@
 <robot name="arrow" xmlns:xacro="http://www.ros.org/wiki/xacro">
 	<xacro:arg name="add_world_link" default="False" />
-	<xacro:property name="color_rgba" default="0.9 0.1 0.1 0.8" />
+	<xacro:arg name="color_rgba" default="1 0 0 1" />
+	<xacro:property name="color_rgba" default="$(arg color_rgba)" />
 	<xacro:property name="add_world_link" default="$(arg add_world_link)" />
-	<material name="red">
-		<color rgba="1 0 0 1"/>
+	<material name="color">
+		<color rgba="${color_rgba}"/>
 	</material>
 	<xacro:macro name="box_inertial" params="mass x y z pose_xyz pose_rpy">
@@ -22,5 +23,5 @@
                 <!-- <mesh filename="package://adarl_envs/models/arrow.stl"  scale="0.001 0.001 0.001"/> -->
             </geometry>
-			<material name="red"/>
+			<material name="color"/>
         </visual>
 		<xacro:box_inertial mass="0.001" x="1" y="1" z="1" pose_xyz="0 0 0" pose_rpy="0 0 0"/>
