Commit message: GraspVecEnv back in working order

File: src/adarl_envs/models/cube.urdf.xacro (robot description, xacro)
@@ -2,19 +2,28 @@
 <robot name="cube" xmlns:xacro="http://www.ros.org/wiki/xacro">
   <xacro:arg name="mass" default="0.1" />
+  <xacro:arg name="size" default="0.06" />
+  <xacro:arg name="red" default="1" />
+  <xacro:arg name="green" default="0.0" />
+  <xacro:arg name="blue" default="0.0" />
+  <xacro:arg name="alpha" default="1.0" />
+  <xacro:arg name="gazebo" default="true" />
+  <xacro:arg name="add_floating_joint" default="true" />
+  <xacro:arg name="add_fixed_joint" default="false" />
+  <xacro:arg name="fixed_joint_xyz" default="0 0 0" />
+  <xacro:arg name="fixed_joint_rpy" default="0 0 0" />
   <xacro:property name="mass" value="$(arg mass)" />
-  <xacro:arg name="size" default="0.06" />
   <xacro:property name="size" value="$(arg size)" />
-  <xacro:arg name="red" default="1" />
   <xacro:property name="red" value="$(arg red)" />
-  <xacro:arg name="green" default="0.0" />
   <xacro:property name="green" value="$(arg green)" />
-  <xacro:arg name="blue" default="0.0" />
   <xacro:property name="blue" value="$(arg blue)" />
-  <xacro:arg name="alpha" default="1.0" />
   <xacro:property name="alpha" value="$(arg alpha)" />
-  <xacro:arg name="gazebo" default="true" />
   <xacro:property name="gazebo" value="$(arg gazebo)" />
-  <xacro:arg name="add_floating_joint" default="true" />
   <xacro:property name="add_floating_joint" value="$(arg add_floating_joint)" />
+  <xacro:property name="add_fixed_joint" value="$(arg add_fixed_joint)" />
+  <xacro:property name="fixed_joint_xyz" value="$(arg fixed_joint_xyz)" />
+  <xacro:property name="fixed_joint_rpy" value="$(arg fixed_joint_rpy)" />
+	<material name="color">
+		<color rgba="${red} ${green} ${blue} ${alpha}"/>
+	</material>
     <xacro:macro name="box_inertial" params="mass x y z pose_xyz pose_rpy">
         <inertial>
@@ -30,4 +39,5 @@
 				<box size="${size} ${size} ${size}"/>
 			</geometry>
+			<material name="color"/>
 	    </visual>
         <collision>
@@ -71,4 +81,12 @@
         </joint>
     </xacro:if>
+    <xacro:if value="${add_fixed_joint}">
+        <link name="world"/>
+        <joint name="fixed_joint" type="fixed">
+            <parent link="world" />
+            <child link="cube" />
+            <origin xyz="${fixed_joint_xyz}" rpy="${fixed_joint_rpy}"/>
+        </joint>
+    </xacro:if>
     <gazebo reference="cube"> <!-- reference to a existing "link" -->
         <visual>

Commit message: grasping works on franka and centauro (no table collision), tuning loco_centauro (SAC)

File: src/adarl_envs/models/cube.urdf.xacro (robot description, xacro)
@@ -12,4 +12,5 @@
   <xacro:arg name="fixed_joint_xyz" default="0 0 0" />
   <xacro:arg name="fixed_joint_rpy" default="0 0 0" />
+  <xacro:arg name="has_collision" default="true" />
   <xacro:property name="mass" value="$(arg mass)" />
   <xacro:property name="size" value="$(arg size)" />
@@ -23,4 +24,5 @@
   <xacro:property name="fixed_joint_xyz" value="$(arg fixed_joint_xyz)" />
   <xacro:property name="fixed_joint_rpy" value="$(arg fixed_joint_rpy)" />
+  <xacro:property name="has_collision" value="$(arg has_collision)" />
 	<material name="color">
 		<color rgba="${red} ${green} ${blue} ${alpha}"/>
@@ -41,10 +43,12 @@
 			<material name="color"/>
 	    </visual>
-        <collision>
-            <origin xyz="0 0 0" rpy="0 0 0"/>
-            <geometry>
-                <box size="${size} ${size} ${size}"/>
-            </geometry>
-        </collision>
+        <xacro:if value="${has_collision}">
+            <collision>
+                <origin xyz="0 0 0" rpy="0 0 0"/>
+                <geometry>
+                    <box size="${size} ${size} ${size}"/>
+                </geometry>
+            </collision>
+        </xacro:if>
         <xacro:box_inertial mass="${mass}" x="0.06" y="0.06" z="0.06" pose_xyz="0 0 0" pose_rpy="0 0 0"/>
         <contact> <!-- for pybullet -->
